Commit message: Update global configuration, model paths, and robot control parameters
- Changed PLAY_DIR in global_config.py to point to a new model file.
- Increased MAX_ITER to 20000 and SAVE_DIV to 1000 for training parameters.
- Removed outdated ONNX model files and added new model files.
- Modified play.py to adjust command values and disable robot pushing.
- Updated TinkerV2 URDF to change base link properties and added a battery link.
- Enhanced sim2sim_tinker.py for keyboard control of robot velocities.
- Updated inference_node.py and rdk_inference.py to use new model paths and added action clipping.
- Added new test scripts for height and distance measurements in the Tinker model.
- Documented planned updates in update_plan.txt for future development.

File: resources/TinkerV2_URDF/urdf/TinkerV2_URDF.urdf (robot description, URDF)
Before this commit: robot TinkerV2_URDF, 11 links, 10 joints
Links:
- added link battery_link, mass 1.0; collision box size=0.04 0.06 0.12; visual box size=0.04 0.06 0.12
- link base_link: mass 3 -> 2.5
Joints:
- added joint battery_joint: type fixed, parent base_link, child battery_link, origin xyz=-0.14 0 0.06 rpy=0 0 0
